File: 01_Microcontroller_Unit_Board/01_Microcontroller_Unit_Board.kicad_sch (KiCad schematic)
At the start: 35 parts, among them J1 10118192-0001LF, J2 TSM-103-01-S-SV, J3 61301811121, J4 61301811121, Q1 BC847BDW1T1G, SW1 B3U-1000P, SW2 B3U-1000P

Commit message: Final check on PCBs, completed on Aug 25, 2026
Parts:
- removed J3, J4: 61301811121, Connector Assemblies:Wurth_61301811121, symbol Connector Assemblies:Wurth_61301811121
- removed L1: 1.5µH(±20%), Inductors:TDK_SPM6530T-1R5M-HZ, symbol Inductors:TDK_SPM6530T-1R5M-HZ
- added C12: 0.1µF(±10%), Capacitors:0402 (1005 Metric), symbol Capacitors:Murata_GCM155R71E104KE02D
- added DAIC1: ADS1115IDGSR, Data Acquisition ICs:10-VSSOP, symbol Data Acquisition ICs:TI_ADS1115IDGSR
- added J3, J4: 61302411121, Connector Assemblies:Wurth_61302411121, symbol Connector Assemblies:Wurth_61302411121
- added L1: 1.5µH(±20%), Inductors:Coilcraft_XFL4020-152MEC, symbol Inductors:Coilcraft_XFL4020-152MEC
- added R13, R14: 10kΩ(±1%), Resistors:0402 (1005 Metric), symbol Resistors:Vishay_CRCW040210K0FKED
- added SW3: CL-SB-12B-01T, Switches:Nidec_CL-SB-12B-01T, symbol Switches:Nidec_CL-SB-12B-01T
- C1, C2, C4: Supplier Price ($) 1.25 -> 1.38
- C10: Manufacturer Part # GCM31CR71E475KA55L -> GCM31CR71E475KA55K; Supplier Part # 490-4794-1-ND -> 490-11168-1-ND; Supplier Price ($) 0.31 -> 0.33
- C11, C3, C8, C9: Supplier Price ($) 0.10 -> 0.11
- C5, C6, C7: Supplier Price ($) 0.64 -> 0.67
- CIIC1: Supplier Price ($) 4.14 -> 5.46
- D1: Supplier Price ($) 0.38 -> 0.64
- D2: Supplier Price ($) 0.47 -> 0.53
- D3: Supplier Price ($) 0.59 -> 1.09
- J1: Supplier Price ($) 0.43 -> 0.50
- J2: Type SMD -> Through Hole
- MCU1: Supplier Price ($) 6.24 -> 6.43
- Q1: Supplier Price ($) 0.18 -> 0.19
Connections:
- net +3V3: now also C12.1, DAIC1.8 (VDD), J3.12, J3.13, R13.1, R14.1
- net EN: now also J3.5
- net GND: now also C12.2, DAIC1.1 (ADDR), DAIC1.3 (GND), J3.17, J3.18, J3.19, J3.20, J4.18, J4.19, J4.20, J4.21, J4.22, J4.23, J4.24, SW3.1
- net GPIO0/ADC2_CH1: now also J4.11
- net GPIO12/ADC2_CH5: now also J4.15
- net GPIO13/ADC2_CH4: now also J4.14
- net GPIO14/ADC2_CH6: now also J4.16
- net GPIO15/ADC2_CH3: now also J4.13
- net GPIO19: now also J4.3
- net GPIO20: now also J4.9
- net GPIO21: now also DAIC1.9 (SDA), J4.1, R14.2
- net GPIO22: now also DAIC1.10 (SCL), J4.2, R13.2
- net GPIO25/ADC2_CH8/DAC_1: now also J3.10
- net GPIO26/ADC2_CH9/DAC_2: now also J3.11
- net GPIO27/ADC2_CH7: now also J4.17
- net GPIO2/ADC2_CH2: now also J4.12
- net GPIO32/ADC1_CH4/XTAL32_IN: now also J3.8
- net GPIO33/ADC1_CH5/XTAL32_OUT: now also J3.9
- net GPIO34/ADC1_CH6: now also J3.6
- net GPIO35/ADC1_CH7: now also J3.7
- net GPIO36/ADC1_CH0: now also J3.1
- net GPIO37/ADC1_CH1: now also J3.2
- net GPIO38/ADC1_CH2: now also J3.3
- net GPIO39/ADC1_CH3: now also J3.4
- net GPIO4/ADC2_CH0: now also J4.10
- net GPIO5: now also J4.6
- net GPIO7: now also J4.8
- net GPIO8: now also J4.7
- net RXD0: now also J4.5
- net TXD0: now also J4.4
- net VBUS: now also J3.15
- net VIN: now also J3.14
- net VUSB: now also J3.16
- net at C3.1, PMIC1.1 (VINA), PMIC1.13 (PS/SYNC): now also SW3.3; no longer PMIC1.12 (EN)
- net at PMIC1.6 (L2), PMIC1.7 (L2): now also L1.1
- net at PMIC1.8 (L1), PMIC1.9 (L1): now also L1.2
- new net: PMIC1.12 (EN), SW3.2
- new net AIN0: DAIC1.4 (AIN0), J3.22
- new net AIN1: DAIC1.5 (AIN1), J3.21
- new net AIN2: DAIC1.6 (AIN2), J3.24
- new net AIN3: DAIC1.7 (AIN3), J3.23
- no-connect marks 16 -> 17
Other:
- moved on the sheet: C10, C11, C5, C6, CIIC1, J2, Q1A, Q1B, R10, R11, R5, R6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
