File: 02_Power_Board/02_Power_Board.kicad_sch (KiCad schematic)
At the start: 120 parts, among them J1 61301811121, J10 NPTC021KFXC-RC, J11 NPTC021KFXC-RC, J12 NPTC021KFXC-RC, J13 NPTC021KFXC-RC, J14 NPTC021KFXC-RC, J15 NPTC021KFXC-RC, J16 NPTC021KFXC-RC, J17 NPTC021KFXC-RC, J18 NPTC021KFXC-RC, J19 NPTC021KFXC-RC, J2 61301811821, J20 61302011821, J21 61302011121, J22 61302011821, J23 61302011121, J3 61301811121, J4 61301811821, J5 1096, J6 TSM-103-01-S-SV, J8 NPTC021KFXC-RC, J9 NPTC021KFXC-RC, Q1 BSS138, Q2 BSS138, Q3 BSS138, Q4 AO3401A, SW1 CL-SB-12A-12T

Commit message: Final check on PCBs, completed on Aug 25, 2026
Parts:
- removed C4: 0.1µF(±10%), Capacitors:0402 (1005 Metric), symbol Capacitors:Murata_GCM155R71E104KE02D
- removed C5, C6: 4.7µF(±10%), Capacitors:1206 (3216 Metric), symbol Capacitors:Murata_GCM31CR71E475KA55L
- removed J1, J3: 61301811121, Connector Assemblies:Wurth_61301811121, symbol Connector Assemblies:Wurth_61301811121
- removed J10, J11, J12, J13, J14, J15, J16, J17, J18, J19, J8, J9: NPTC021KFXC-RC, Connector Assemblies:Sullins_NPTC021KFXC-RC, symbol Connector Assemblies:Sullins_NPTC021KFXC-RC
- removed J2, J4: 61301811821, Connector Assemblies:Wurth_61301811821, symbol Connector Assemblies:Wurth_61301811821
- removed PMIC2: TPS22919DCKR, Power Management ICs:SOT-363, symbol Power Management ICs:TI_TPS22919DCKR
- removed R16: 1Ω(±1%), Resistors:2512 (6332 Metric), symbol Resistors:Isabellenhuette_SMS-1R00-1.0
- removed R19, R20: 15kΩ(±1%), Resistors:0402 (1005 Metric), symbol Resistors:Vishay_CRCW040215K0FKED
- removed R21: 47kΩ(±1%), Resistors:0402 (1005 Metric), symbol Resistors:Vishay_CRCW040247K0FKED
- removed R22: 100kΩ(±1%), Resistors:0402 (1005 Metric), symbol Resistors:Vishay_CRCW0402100KFKED
- removed R23: 453Ω(±1%), Resistors:0402 (1005 Metric), symbol Resistors:Vishay_CRCW0402453RFKED
- removed R27: 97.6kΩ(±1%), Resistors:0402 (1005 Metric), symbol Resistors:Vishay_CRCW040297K6FKED
- removed R28: 88.7kΩ(±1%), Resistors:0402 (1005 Metric), symbol Resistors:Vishay_CRCW040288K7FKED
- removed SW1: CL-SB-12A-12T, Switches:Nidec_CL-SB-12A-12T, symbol Switches:Nidec_CL-SB-12A-12T
- removed TP4: 5019, Test Points:Keystone_5019, symbol Test Points:Keystone_5019
- added C4: 1µF(±10%), Capacitors:0603 (1608 Metric), symbol Capacitors:Murata_GCM188R71E105KA64D
- added J1, J3: 61302411121, Connector Assemblies:Wurth_61302411121, symbol Connector Assemblies:Wurth_61302411121
- added J10, J11, J12, J13, J14, J15, J16, J17, J18, J19, J8, J9: PSS-02-01-T-S, Connector Assemblies:Samtec_PSS-02-01-T-S, symbol Connector Assemblies:Samtec_PSS-02-01-T-S
- added J2, J4: PPTC241LFBN-RC, Connector Assemblies:Sullins_PPTC241LFBN-RC, symbol Connector Assemblies:Sullins_PPTC241LFBN-RC
- added R16: 100mΩ(±0.1%), Resistors:2512 (6332 Metric), symbol Resistors:Ohmite_PCS2512DR1000ET
- added R19, R20, R22: 30kΩ(±1%), Resistors:0402 (1005 Metric), symbol Resistors:Vishay_CRCW040230K0FKED
- added R21: 12kΩ(±1%), Resistors:0402 (1005 Metric), symbol Resistors:Vishay_CRCW040212K0FKED
- added R27: 91kΩ(±1%), Resistors:0402 (1005 Metric), symbol Resistors:Vishay_CRCW040291K0FKED
- added R28: 82.5kΩ(±1%), Resistors:0402 (1005 Metric), symbol Resistors:Vishay_CRCW040282K5FKED
- C1, C15, C16, C3: Manufacturer Part # GCM31CR71E475KA55L -> GCM31CR71E475KA55K; Supplier Part # 490-4794-1-ND -> 490-11168-1-ND; Supplier Price ($) 0.31 -> 0.33
- C10, C14, C9: Supplier Price ($) 0.4 -> 0.43
- C11, C21, C26: Supplier Price ($) 0.20 -> 0.19
- C12, C17, C20, C25, C7: Supplier Price ($) 0.10 -> 0.11
- C13, C19, C8: Manufacturer Part # GCM155R71E103KA37D -> GCM155R71E103KA37J; Supplier Part # 490-6043-1-ND -> 490-GCM155R71E103KA37JCT-ND; Supplier Price ($) 0.10 -> 0.11
- C2: Subcategory Surface Mount Think Film Capacitor -> Surface Mount MLCC; Supplier Price ($) 0.64 -> 0.67
- D2: value Wurth_150060BS75000 -> 150060BS75000; Supplier Price ($) 0.17 -> 0.16
- D5, D6: value BAT760-7 -> CUS10S30,H3F; Manufacturer Diodes Incorporated -> Toshiba Semiconductor and Storage; Manufacturer Part # BAT760-7 -> CUS10S30,H3F; Short Description DIODE SCHOTTKY 30V 1A SOD323 -> DIODE SCHOTTKY 30V 1A USC; Supplier Part # BAT760DICT-ND -> CUS10S30H3FCT-ND; Supplier Price ($) 0.47 -> 0.36
- J5: Type SMD -> Hybrid
- L1, L2: Supplier Part # 732-1175-1-ND -> 495-77086-1-ND; Supplier Price ($) 1.59 -> 1.76
- OPA1: Supplier Price ($) 1.67 -> 1.72
- PMIC3: Supplier Price ($) 0.33 -> 0.34
- PMIC4: Supplier Price ($) 1.29 -> 1.45
- PMIC5: Supplier Price ($) 4.00 -> 4.93
- PMIC6: value TPS65131RGER -> TPS65131RGET; Manufacturer Part # TPS65131RGER -> TPS65131RGET; Supplier Part # 296-41760-1-ND -> 296-17349-1-ND; Supplier Price ($) 3.51 -> 4.64
- PMIC7: Supplier Price ($) 0.43 -> 0.46
- PMIC8: Supplier Price ($) 0.47 -> 0.51
- Q1, Q2, Q3: Supplier Price ($) 0.28 -> 0.32
- R24: Short Description RES 100 OHM 1% 1/10W 0402 -> RES 100 OHM 1% 1/16W 0402
- R3: Short Description RES 976 OHM 1% 1/10W 0402 -> RES 976 OHM 1% 1/16W 0402
Connections:
- net VSYS is gone; now on net VIN: J6.2, Q4.2
- net +2V5: now also J1.21, J2.21
- net +3V3: now also J20.7, J21.7, J22.11, J23.11, OPA1.8, C4.1, J1.12, J1.13, J2.12, J2.13
- net EN: now also J1.5, J2.5
- net GND: now also J20.13, J20.14, J20.15, J21.13, J21.14, J21.15, C4.2, J1.17, J1.18, J1.19, J1.20, J11.2, J13.2, J15.2, J17.2, J19.2, J2.17, J2.18, J2.19, J2.20, J3.18, J3.19, J3.20, J3.21, J3.22, J3.23, J3.24, J4.18, J4.19, J4.20, J4.21, J4.22, J4.23, J4.24, J9.2, R20.2, R22.2, R27.2
- net GPIO0/ADC2_CH1: now also J3.11, J4.11
- net GPIO12/ADC2_CH5: now also J3.15, J4.15; no longer J20.9, J21.9
- net GPIO13/ADC2_CH4: now also J3.14, J4.14
- net GPIO14/ADC2_CH6: now also J20.9, J21.9, J3.16, J4.16; no longer J20.8, J21.8
- net GPIO15/ADC2_CH3: now also J3.13, J4.13; no longer J20.13, J21.13
- net GPIO19: now also J22.15, J23.15, J3.3, J4.3
- net GPIO20: now also J3.9, J4.9
- net GPIO21: now also J3.1, J4.1; no longer J20.15, J21.15
- net GPIO22: now also J3.2, J4.2; no longer J20.14, J21.14
- net GPIO25/ADC2_CH8/DAC_1: now also J1.10, J2.10
- net GPIO26/ADC2_CH9/DAC_2: now also J1.11, J2.11
- net GPIO27/ADC2_CH7: now also J20.8, J21.8, J3.17, J4.17; no longer J20.7, J21.7
- net GPIO2/ADC2_CH2: now also J3.12, J4.12; no longer J22.11, J23.11
- net GPIO32/ADC1_CH4/XTAL32_IN: now also J22.12, J23.12, J1.8, J2.8; no longer Q1.3, R4.1
- net GPIO33/ADC1_CH5/XTAL32_OUT: now also J22.13, J23.13, J1.9, J2.9; no longer Q2.3, R6.1
- net GPIO34/ADC1_CH6: now also Q1.3, R4.1, J1.6, J2.6; no longer J20.18, J21.18
- net GPIO35/ADC1_CH7: now also Q2.3, R6.1, J1.7, J2.7; no longer Q3.3, R8.1
- net GPIO39/ADC1_CH3: now also Q3.3, R8.1, J1.4, J2.4
- net GPIO4/ADC2_CH0: now also J22.14, J23.14, J3.10, J4.10; no longer J22.12, J23.12
- net GPIO5: now also J3.6, J4.6; no longer J22.15, J23.15
- net GPIO7: now also J3.8, J4.8; no longer J22.13, J23.13
- net GPIO8: now also J3.7, J4.7; no longer J22.14, J23.14
- net RXD0: now also J3.5, J4.5
- net TXD0: now also J3.4, J4.4
- net VBAT: now also R21.1; no longer OPA1.8
- net VBUS: now also J1.15, J2.15
- net VCHGR_NEG: now also R16.1
- net VCHGR_POS: now also R16.2
- net VIN: now also J1.14, J2.14
- net VUSB: now also J1.16, J2.16
- net at C18.2, PMIC6.22 (FBP), R26.2: now also R27.1
- net at OPA1.3, R18.2: now also R20.1
- net at C12.2, PMIC5.2 (IN), PMIC5.3 (EN)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: now also J10.1, J8.2, J9.1
- net at D5.K, PMIC6.23 (VPOS), R25.2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: now also J12.1
- net at C20.2, PMIC7.1 (IN), TP11.1: now also J12.2, J13.1, J14.1
- net at D6.A, PMIC6.15 (VNEG), R29.1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: now also J16.1
- net at C25.2, PMIC8.2 (IN), TP13.1: now also J16.2, J17.1, J18.1
- net at OPA1.5: now also R21.2, R22.1
- net at PMIC4.1 (VOUT): now also J8.1
- net at C24.2, PMIC6.16 (FBN), R29.2: now also R28.2
- net at C23.1, PMIC6.17 (VREF): now also R28.1
- net at OPA1.2, R17.2: now also R19.2
- net GPIO36/ADC1_CH0 renamed AIN3
- net AIN3: now also J1.1, J1.23, J2.1, J2.23
- net GPIO37/ADC1_CH1 renamed AIN2
- net AIN2: now also J1.2, J1.24, J2.2, J2.24, R19.1
- new net: J10.2, J11.1
- new net: J18.2, J19.1
- new net: J14.2, J15.1
- new net AIN0: J1.22, J1.3, J2.22, J2.3, J20.18, J21.18
Other:
- note added: "+2V5 REGULATION"
- note added: "-2V5 REGULATION"
- note added: "±12V REGULATION"
- note removed: "+2V5 RAIL"
- note removed: "-2V5 RAIL"
- note removed: "SYSTEM VOLTAGE ENABLE"
- note removed: "±12V RAILS"
- moved on the sheet: J20, J21, J22, J23, J6, MH1, MH2, MH3, MH4, OPA1A, OPA1B, R17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
