File: 03_Analog_Front_End_Board/03_Analog_Front_End_Board.kicad_sch (KiCad schematic)
At the start: 115 parts, among them J1 61302011121, J2 61302011121, J3 NPTC021KFXC-RC, J4 NPTC021KFXC-RC, J5 0541043631, J6 TSW-105-07-G-T, J7 TSW-104-07-G-T, Q1 BSS138, Q2 BSS138, Q3 BSS138, Q4 BSS138, Q5 BSS138, Q6 BSS138, Q7 BSS138, Q8 BSS138, Q9 BSS138

Commit message: Final check on PCBs, completed on Aug 25, 2026
Parts:
- removed C27: 0.1µF(±10%), Capacitors:0402 (1005 Metric), symbol Capacitors:Murata_GCM155R71E104KE02D
- removed DAIC1: ADS1115IDGSR, Data Acquisition ICs:10-VSSOP, symbol Data Acquisition ICs:TI_ADS1115IDGSR
- removed R39, R40, R41, R42: 100kΩ(±1%), Resistors:0402 (1005 Metric), symbol Resistors:Vishay_CRCW040266K5FKED
- removed R43, R44, R45: 10kΩ(±1%), Resistors:0402 (1005 Metric), symbol Resistors:Vishay_CRCW040210K0FKED
- added R39, R40, R41, R42: 100kΩ(±1%), Resistors:0402 (1005 Metric), symbol Resistors:Vishay_CRCW0402100KFKED
- C1, C18, C19, C2, C20, C21, C22, C23, C24, C25, C26, C3, C4, C5: Supplier Price ($) 0.20 -> 0.19
- C10, C11, C12, C6, C7, C8, C9: Supplier Price ($) 0.14 -> 0.15
- C15: Supplier Price ($) 0.14 -> 0.13
- C17: Supplier Price ($) 0.13 -> 0.14
- J3, J4: Supplier Price ($) 0.51 -> 0.57
- MUX1: Supplier Price ($) 12.72 -> 13.10
- OPA2: value OPA2192IDGKR -> OPA2192IDGKT; Manufacturer Part # OPA2192IDGKR -> OPA2192IDGKT; Supplier DigiKey -> Mouser; Supplier Part # 296-44480-1-ND -> 595-OPA2192IDGKT; Supplier Price ($) 4.78 -> 6.23
- OPA4: Supplier Price ($) 5.55 -> 6.22
- Q1, Q2, Q3, Q4, Q5, Q6, Q7, Q8, Q9: Supplier Price ($) 0.28 -> 0.32
- R10, R5, R6, R9: Short Description RES 73.2K OHM 1% 1/10W 0402 -> RES 73.2K OHM 1% 1/16W 0402
- R30: Supplier Price ($) 7.57 -> 7.69
Connections:
- net ALERT is gone; now on net GND: J1.13
- net SCL is gone; now on net GND: J1.14
- net SDA is gone; now on net GND: J1.15
- net +1V65: now also R40.1
- net GND: now also R42.1
- net TIA_OUT: now also R41.2
- net at OPA5.4, R38.1, TP15.1: now also R39.1
- net at OPA6.3: now also R41.1, R42.2
- net at OPA6.1: now also R39.2, R40.2
Other:
- note removed: "EXTERNAL ADC"
